File: src/flash.kicad_pcb (KiCad board)
At the start: 2 copper layers, 31 x 29 mm, 5 parts, among them J1 Conn_01x06, J2 Conn_01x06, U2 W25Q128JVS

Commit message: feat: prepare for prod
Routing:
- net GND: track 22.5 -> 139.0 mm, vias 0 -> 4
Other:
- board size 31 x 29 mm -> 45 x 40 mm
Changed lines of the file:
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@@
 		)
 	)
+	(gr_poly
+		(pts
+			(xy 144 74) (xy 153 74) (xy 153 34) (xy 144 34)
+		)
+		(stroke
+			(width 0.2)
+			(type solid)
+		)
+		(fill solid)
+		(layer "F.Cu")
+		(net 2)
+	)
 	(gr_rect
-		(start 156 39)
-		(end 187 68)
+		(start 144 34)
+		(end 189 74)
 		(stroke
 			(width 0.05)
@@
 	)
 	(segment
+		(start 187.5 35.5)
+		(end 148.5 35.5)
+		(width 2)
+		(layer "F.Cu")
+		(net 2)
+	)
+	(segment
 		(start 175.255 64.008)
 		(end 165.766 64.008)
@@
 	)
 	(segment
+		(start 187.5 72.5)
+		(end 147 72.5)
+		(width 2)
+		(layer "F.Cu")
+		(net 2)
+	)
+	(segment
 		(start 174.752 56.222)
 		(end 174.752 60.452)
@@
 		(end 165.528 64.086)
 		(width 0.5)
+		(layer "F.Cu")
+		(net 2)
+	)
+	(segment
+		(start 187.5 35.5)
+		(end 187.5 72.5)
+		(width 2)
 		(layer "F.Cu")
 		(net 2)
@@
 		(net 2)
 	)
+	(via
+		(at 187.5 69)
+		(size 2)
+		(drill 1)
+		(layers "F.Cu" "B.Cu")
+		(teardrops
+			(best_length_ratio 0.5)
+			(max_length 1)
+			(best_width_ratio 1)
+			(max_width 2)
+			(curve_points 0)
+			(filter_ratio 0.9)
+			(enabled no)
+			(allow_two_segments no)
+			(prefer_zone_connections yes)
+		)
+		(net 2)
+	)
+	(via
+		(at 152 69)
+		(size 2)
+		(drill 1)
+		(layers "F.Cu" "B.Cu")
+		(teardrops
+			(best_length_ratio 0.5)
+			(max_length 1)
+			(best_width_ratio 1)
+			(max_width 2)
+			(curve_points 0)
+			(filter_ratio 0.9)
+			(enabled no)
+			(allow_two_segments no)
+			(prefer_zone_connections yes)
+		)
+		(net 2)
+	)
+	(via
+		(at 152 39.5)
+		(size 2)
+		(drill 1)
+		(layers "F.Cu" "B.Cu")
+		(teardrops
+			(best_length_ratio 0.5)
+			(max_length 1)
+			(best_width_ratio 1)
+			(max_width 2)
+			(curve_points 0)
+			(filter_ratio 0.9)
+			(enabled no)
+			(allow_two_segments no)
+			(prefer_zone_connections yes)
+		)
+		(net 2)
+	)
+	(via
+		(at 187.5 39.5)
+		(size 2)
+		(drill 1)
+		(layers "F.Cu" "B.Cu")
+		(teardrops
+			(best_length_ratio 0.5)
+			(max_length 1)
+			(best_width_ratio 1)
+			(max_width 2)
+			(curve_points 0)
+			(filter_ratio 0.9)
+			(enabled no)
+			(allow_two_segments no)
+			(prefer_zone_connections yes)
+		)
+		(net 2)
+	)
